File: arduino-blinky.sch (KiCad schematic (older format))
At the start: 14 parts, among them IC1 ATMEGA8-P, Y1 16 MHz

Commit message: PCB created
Parts:
- D1, D2, D3, D4, D5, D6: footprint (none) -> LEDs:LED_D3.0mm
- IC1: footprint DIL28 -> Housings_DIP:DIP-28_W7.62mm_Socket
Changed lines of the file:
@@
 F 0 "IC1" H 4950 5350 50  0000 L BNN
 F 1 "ATMEGA8-P" H 6200 2600 50  0000 L BNN
-F 2 "DIL28" H 5700 4050 50  0000 C CIN
+F 2 "Housings_DIP:DIP-28_W7.62mm_Socket" H 5700 4050 50  0001 C CIN
 F 3 "" H 5700 4050 50  0000 C CNN
 	1    5700 4050
@@
 $EndComp
 $Comp
-L +5V #PWR5
+L +5V #PWR01
 U 1 1 58C19A29
 P 5700 2650
-F 0 "#PWR5" H 5700 2500 50  0001 C CNN
+F 0 "#PWR01" H 5700 2500 50  0001 C CNN
 F 1 "+5V" H 5700 2790 50  0000 C CNN
 F 2 "" H 5700 2650 50  0000 C CNN
@@
 $EndComp
 $Comp
-L GND #PWR6
+L GND #PWR02
 U 1 1 58C19A90
 P 5700 5550
-F 0 "#PWR6" H 5700 5300 50  0001 C CNN
+F 0 "#PWR02" H 5700 5300 50  0001 C CNN
 F 1 "GND" H 5700 5400 50  0000 C CNN
 F 2 "" H 5700 5550 50  0000 C CNN
@@
 $EndComp
 $Comp
-L +5V #PWR2
+L +5V #PWR03
 U 1 1 58C19B38
 P 4350 2950
-F 0 "#PWR2" H 4350 2800 50  0001 C CNN
+F 0 "#PWR03" H 4350 2800 50  0001 C CNN
 F 1 "+5V" H 4350 3090 50  0000 C CNN
 F 2 "" H 4350 2950 50  0000 C CNN
@@
 $EndComp
 $Comp
-L GND #PWR4
+L GND #PWR04
 U 1 1 58C19BBF
 P 4700 3350
-F 0 "#PWR4" H 4700 3100 50  0001 C CNN
+F 0 "#PWR04" H 4700 3100 50  0001 C CNN
 F 1 "GND" H 4700 3200 50  0000 C CNN
 F 2 "" H 4700 3350 50  0000 C CNN
@@
 $EndComp
 $Comp
-L +5V #PWR3
+L +5V #PWR05
 U 1 1 58C19C11
 P 4600 3250
-F 0 "#PWR3" H 4600 3100 50  0001 C CNN
+F 0 "#PWR05" H 4600 3100 50  0001 C CNN
 F 1 "+5V" H 4600 3390 50  0000 C CNN
 F 2 "" H 4600 3250 50  0000 C CNN
@@
 $EndComp
 $Comp
-L GND #PWR1
+L GND #PWR06
 U 1 1 58C19F80
 P 3300 3800
-F 0 "#PWR1" H 3300 3550 50  0001 C CNN
+F 0 "#PWR06" H 3300 3550 50  0001 C CNN
 F 1 "GND" H 3300 3650 50  0000 C CNN
 F 2 "" H 3300 3800 50  0000 C CNN
@@
 $EndComp
 $Comp
-L GND #PWR7
+L GND #PWR07
 U 1 1 58C1A632
 P 5750 2050
-F 0 "#PWR7" H 5750 1800 50  0001 C CNN
+F 0 "#PWR07" H 5750 1800 50  0001 C CNN
 F 1 "GND" H 5750 1900 50  0000 C CNN
 F 2 "" H 5750 2050 50  0000 C CNN
@@
 $EndComp
 $Comp
-L +5V #PWR8
+L +5V #PWR08
 U 1 1 58C1A875
 P 6200 1700
-F 0 "#PWR8" H 6200 1550 50  0001 C CNN
+F 0 "#PWR08" H 6200 1550 50  0001 C CNN
 F 1 "+5V" H 6200 1840 50  0000 C CNN
 F 2 "" H 6200 1700 50  0000 C CNN
@@
 F 0 "D1" H 7450 3500 50  0000 C CNN
 F 1 "LED" H 7450 3300 50  0000 C CNN
-F 2 "" H 7450 3400 50  0000 C CNN
+F 2 "LEDs:LED_D3.0mm" H 7450 3400 50  0001 C CNN
 F 3 "" H 7450 3400 50  0000 C CNN
 	1    7450 3400
@@
 F 0 "D2" H 7450 3800 50  0000 C CNN
 F 1 "LED" H 7450 3600 50  0000 C CNN
-F 2 "" H 7450 3700 50  0000 C CNN
+F 2 "LEDs:LED_D3.0mm" H 7450 3700 50  0001 C CNN
 F 3 "" H 7450 3700 50  0000 C CNN
 	1    7450 3700
@@
 F 0 "D3" H 7450 4100 50  0000 C CNN
 F 1 "LED" H 7450 3900 50  0000 C CNN
-F 2 "" H 7450 4000 50  0000 C CNN
+F 2 "LEDs:LED_D3.0mm" H 7450 4000 50  0001 C CNN
 F 3 "" H 7450 4000 50  0000 C CNN
 	1    7450 4000
@@
 F 0 "D4" H 7450 5100 50  0000 C CNN
 F 1 "LED" H 7450 4900 50  0000 C CNN
-F 2 "" H 7450 5000 50  0000 C CNN
+F 2 "LEDs:LED_D3.0mm" H 7450 5000 50  0001 C CNN
 F 3 "" H 7450 5000 50  0000 C CNN
 	1    7450 5000
@@
 F 0 "D5" H 7450 5400 50  0000 C CNN
 F 1 "LED" H 7450 5200 50  0000 C CNN
-F 2 "" H 7450 5300 50  0000 C CNN
+F 2 "LEDs:LED_D3.0mm" H 7450 5300 50  0001 C CNN
 F 3 "" H 7450 5300 50  0000 C CNN
 	1    7450 5300
@@
 F 0 "D6" H 7450 5700 50  0000 C CNN
 F 1 "LED" H 7450 5500 50  0000 C CNN
-F 2 "" H 7450 5600 50  0000 C CNN
+F 2 "LEDs:LED_D3.0mm" H 7450 5600 50  0001 C CNN
 F 3 "" H 7450 5600 50  0000 C CNN
 	1    7450 5600
@@
 $EndComp
 $Comp
-L GND #PWR10
+L GND #PWR09
 U 1 1 58C1B696
 P 8350 3700
-F 0 "#PWR10" H 8350 3450 50  0001 C CNN
+F 0 "#PWR09" H 8350 3450 50  0001 C CNN
 F 1 "GND" H 8350 3550 50  0000 C CNN
 F 2 "" H 8350 3700 50  0000 C CNN
@@
 $EndComp
 $Comp
-L GND #PWR9
+L GND #PWR010
 U 1 1 58C1B6C6
 P 8300 5300
-F 0 "#PWR9" H 8300 5050 50  0001 C CNN
+F 0 "#PWR010" H 8300 5050 50  0001 C CNN
 F 1 "GND" H 8300 5150 50  0000 C CNN
 F 2 "" H 8300 5300 50  0000 C CNN
